Commit message: Restructured simulation package

File: dataset_gen/src/camera_controls/urdf/camera.urdf.xacro (robot description, xacro)
@@ -2,4 +2,9 @@
 <robot xmlns:xacro="http://www.ros.org/wiki/xacro" name="camera">
   <link name="camera">
+    <visual>
+      <geometry>
+        <box size="0.025 0.025 0.025"/>
+      </geometry>
+    </visual>
     <inertial>
       <origin xyz="0 0 0" rpy="0 0 0" />
@@ -8,5 +13,27 @@
     </inertial>
   </link>
+  <link name="drone">
+    <visual>
+      <geometry>
+        <sphere radius="0.05"/>
+      </geometry>
+    <origin xyz="0 0 0" rpy="0 0 0" />
+    </visual>
+    <inertial>
+      <origin xyz="0 0 0" rpy="0 0 0" />
+      <mass value="1" />
+      <inertia ixx="1" ixy="0" ixz="0" iyy="1" iyz="0" izz="1" />
+    </inertial>
+  </link>
+  <joint name="drone_to_camera" type="fixed">
+    <parent link="drone"/>
+    <child link="camera"/>
+    <origin xyz="0.05 0 0"/>
+  </joint>
+  <gazebo reference="drone">
+    <material>Gazebo/Red</material>
+  </gazebo>
   <gazebo reference="camera">
+    <material>Gazebo/Blue</material>
     <sensor type="camera" name="camera">
       <update_rate>30.0</update_rate>

File: dataset_gen/src/camera_controls/urdf/camera_small.urdf.xacro (robot description, xacro)
@@ -2,4 +2,9 @@
 <robot xmlns:xacro="http://www.ros.org/wiki/xacro" name="camera">
   <link name="camera">
+    <visual>
+      <geometry>
+        <box size="0.025 0.025 0.025"/>
+      </geometry>
+    </visual>
     <inertial>
       <origin xyz="0 0 0" rpy="0 0 0" />
@@ -8,5 +13,27 @@
     </inertial>
   </link>
+  <link name="drone">
+    <visual>
+      <geometry>
+        <sphere radius="0.05"/>
+      </geometry>
+    <origin xyz="0 0 0" rpy="0 0 0" />
+    </visual>
+    <inertial>
+      <origin xyz="0 0 0" rpy="0 0 0" />
+      <mass value="1" />
+      <inertia ixx="1" ixy="0" ixz="0" iyy="1" iyz="0" izz="1" />
+    </inertial>
+  </link>
+  <joint name="drone_to_camera" type="fixed">
+    <parent link="drone"/>
+    <child link="camera"/>
+    <origin xyz="0.05 0 0"/>
+  </joint>
+  <gazebo reference="drone">
+    <material>Gazebo/Red</material>
+  </gazebo>
   <gazebo reference="camera">
+    <material>Gazebo/Blue</material>
     <sensor type="camera" name="camera">
       <update_rate>30.0</update_rate>

File: dataset_gen/src/simulation/urdf/bulding.urdf.xacro (robot description, xacro)
@@ -9,5 +9,5 @@
       <origin xyz="0 -5 0" rpy="0 0 0" />
       <geometry>
-        <mesh filename="package://cottage/meshes/bulding.dae" scale="2 2 2" />
+        <mesh filename="package://simulation/meshes/bulding.dae" scale="2 2 2" />
       </geometry>
     </visual>
@@ -15,5 +15,5 @@
       <origin xyz="0 -5 0" rpy="0 0 0" />
       <geometry>
-        <mesh filename="package://cottage/meshes/bulding.dae" scale="2 2 2" />
+        <mesh filename="package://simulation/meshes/bulding.dae" scale="2 2 2" />
       </geometry>
     </collision>

File: dataset_gen/src/simulation/urdf/cottage_blender_Cube.urdf.xacro (robot description, xacro)
@@ -1,4 +1,4 @@
 <robot name="robot">
-  <link name="cottage_blender_ground_link">
+  <link name="cottage_blender_Cube_link">
     <inertial>
       <origin xyz="0 0 0" rpy="0 0 0" />
@@ -9,5 +9,5 @@
       <origin xyz="0 0 0" rpy="0 0 0" />
       <geometry>
-        <mesh filename="package://cottage/meshes/cottage_blender_ground.dae" />
+        <mesh filename="package://simulation/meshes/cottage_blender_Cube.dae" />
       </geometry>
     </visual>
@@ -15,10 +15,10 @@
       <origin xyz="0 0 0" rpy="0 0 0" />
       <geometry>
-        <mesh filename="package://cottage/meshes/cottage_blender_ground.dae" />
+        <mesh filename="package://simulation/meshes/cottage_blender_Cube.dae" />
       </geometry>
     </collision>
   </link>
-  <gazebo reference="cottage_blender_ground_link">
-    <material>grass</material>
+  <gazebo reference="cottage_blender_Cube_link">
+    <material>cottage_texture</material>
   </gazebo>
   <gazebo> <static>true</static></gazebo>

File: dataset_gen/src/simulation/urdf/cottage_blender_ground.urdf.xacro (robot description, xacro)
@@ -1,4 +1,4 @@
 <robot name="robot">
-  <link name="cottage_blender_light_3_link">
+  <link name="cottage_blender_ground_link">
     <inertial>
       <origin xyz="0 0 0" rpy="0 0 0" />
@@ -9,5 +9,5 @@
       <origin xyz="0 0 0" rpy="0 0 0" />
       <geometry>
-        <mesh filename="package://cottage/meshes/cottage_blender_light_3.dae" />
+        <mesh filename="package://simulation/meshes/cottage_blender_ground.dae" />
       </geometry>
     </visual>
@@ -15,8 +15,11 @@
       <origin xyz="0 0 0" rpy="0 0 0" />
       <geometry>
-        <mesh filename="package://cottage/meshes/cottage_blender_light_3.dae" />
+        <mesh filename="package://simulation/meshes/cottage_blender_ground.dae" />
       </geometry>
     </collision>
   </link>
+  <gazebo reference="cottage_blender_ground_link">
+    <material>grass</material>
+  </gazebo>
   <gazebo> <static>true</static></gazebo>
 </robot>

File: dataset_gen/src/simulation/urdf/cottage_blender_light_1.urdf.xacro (robot description, xacro)
@@ -9,5 +9,5 @@
       <origin xyz="0 0 0" rpy="0 0 0" />
       <geometry>
-        <mesh filename="package://cottage/meshes/cottage_blender_light_1.dae" />
+        <mesh filename="package://simulation/meshes/cottage_blender_light_1.dae" />
       </geometry>
     </visual>
@@ -15,5 +15,5 @@
       <origin xyz="0 0 0" rpy="0 0 0" />
       <geometry>
-        <mesh filename="package://cottage/meshes/cottage_blender_light_1.dae" />
+        <mesh filename="package://simulation/meshes/cottage_blender_light_1.dae" />
       </geometry>
     </collision>

File: dataset_gen/src/simulation/urdf/cottage_blender_light_2.urdf.xacro (robot description, xacro)
@@ -1,4 +1,4 @@
 <robot name="robot">
-  <link name="cottage_blender_Cube_link">
+  <link name="cottage_blender_light_2_link">
     <inertial>
       <origin xyz="0 0 0" rpy="0 0 0" />
@@ -9,5 +9,5 @@
       <origin xyz="0 0 0" rpy="0 0 0" />
       <geometry>
-        <mesh filename="package://cottage/meshes/cottage_blender_Cube.dae" />
+        <mesh filename="package://simulation/meshes/cottage_blender_light_2.dae" />
       </geometry>
     </visual>
@@ -15,11 +15,8 @@
       <origin xyz="0 0 0" rpy="0 0 0" />
       <geometry>
-        <mesh filename="package://cottage/meshes/cottage_blender_Cube.dae" />
+        <mesh filename="package://simulation/meshes/cottage_blender_light_2.dae" />
       </geometry>
     </collision>
   </link>
-  <gazebo reference="cottage_blender_Cube_link">
-    <material>cottage_texture</material>
-  </gazebo>
   <gazebo> <static>true</static></gazebo>
 </robot>

File: dataset_gen/src/simulation/urdf/cottage_blender_light_3.urdf.xacro (robot description, xacro)
@@ -1,4 +1,4 @@
 <robot name="robot">
-  <link name="cottage_blender_light_2_link">
+  <link name="cottage_blender_light_3_link">
     <inertial>
       <origin xyz="0 0 0" rpy="0 0 0" />
@@ -9,5 +9,5 @@
       <origin xyz="0 0 0" rpy="0 0 0" />
       <geometry>
-        <mesh filename="package://cottage/meshes/cottage_blender_light_2.dae" />
+        <mesh filename="package://simulation/meshes/cottage_blender_light_3.dae" />
       </geometry>
     </visual>
@@ -15,5 +15,5 @@
       <origin xyz="0 0 0" rpy="0 0 0" />
       <geometry>
-        <mesh filename="package://cottage/meshes/cottage_blender_light_2.dae" />
+        <mesh filename="package://simulation/meshes/cottage_blender_light_3.dae" />
       </geometry>
     </collision>
